Commit message: update mybot description

File: mybot_description/urdf/mybot.xacro (robot description, xacro)
@@ -1,113 +1,84 @@
 <?xml version='1.0'?>
 <robot name="myrobot" xmlns:xacro="http://www.ros.org/wiki/xacro">
-  <xacro:include filename="$(find mybot_description)/urdf/mybot.gazebo" />
-  <link name='chassis'>
-    <pose>0 0 0.1 0 0 0</pose>
-    <inertial>
-      <mass value="10.0"/>
-      <origin xyz="0.0 0 0.1" rpy=" 0 0 0"/>
-      <inertia
-          ixx="0.5" ixy="0" ixz="0"
-          iyy="1.0" iyz="0"
-          izz="0.1"
-      />
-    </inertial>
-    <collision name='collision'>
-      <geometry>
-        <box size=".4 .2 .1"/>
-      </geometry>
-    </collision>
-    <visual name='chassis_visual'>
-      <origin xyz="0 0 0" rpy=" 0 0 0"/>
-      <geometry>
-        <box size=".4 .2 .1"/>
-      </geometry>
-    </visual>
-    <collision name='caster_collision'>
-      <origin xyz="-0.15 0 -0.05" rpy=" 0 0 0"/>
-      <geometry>
-        <sphere radius="0.05"/>
-      </geometry>
-      <surface>
-        <friction>
-          <ode>
-            <mu>0</mu>
-            <mu2>0</mu2>
-            <slip1>1.0</slip1>
-            <slip2>1.0</slip2>
-          </ode>
-        </friction>
-      </surface>
-    </collision>
-    <visual name='caster_visual'>
-      <origin xyz="-0.15 0 -0.05" rpy=" 0 0 0"/>
-      <geometry>
-        <sphere radius="0.05"/>
-      </geometry>
-    </visual>
-  </link>
-  <link name="left_wheel">
-    <!--origin xyz="0.1 0.13 0.1" rpy="0 1.5707 1.5707"/-->
-    <collision name="collision">
-      <origin xyz="0 0 0" rpy="0 1.5707 1.5707"/>
-      <geometry>
-        <cylinder radius="0.1" length="0.05"/>
-      </geometry>
-    </collision>
-    <visual name="left_wheel_visual">
-      <origin xyz="0 0 0" rpy="0 1.5707 1.5707"/>
-      <geometry>
-        <cylinder radius="0.1" length="0.05"/>
-      </geometry>
-    </visual>
-    <inertial>
-      <origin xyz="0 0 0" rpy="0 1.5707 1.5707"/>
-      <mass value="5"/>
-      <cylinder_inertia m="5" r="0.1" h="0.05"/>
-      <inertia
-        ixx="1.0" ixy="0.0" ixz="0.0"
-        iyy="1.0" iyz="0.0"
-        izz="1.0"/>
-    </inertial>
-  </link>
-  <link name="right_wheel">
-    <!--origin xyz="0.1 -0.13 0.1" rpy="0 1.5707 1.5707"/-->
-    <collision name="collision">
-      <origin xyz="0 0 0" rpy="0 1.5707 1.5707"/>
-      <geometry>
-        <cylinder radius="0.1" length="0.05"/>
-      </geometry>
-    </collision>
-    <visual name="right_wheel_visual">
-      <origin xyz="0 0 0" rpy="0 1.5707 1.5707"/>
-      <geometry>
-        <cylinder radius="0.1" length="0.05"/>
-      </geometry>
-    </visual>
-    <inertial>
-      <origin xyz="0 0 0" rpy="0 1.5707 1.5707"/>
-      <mass value="5"/>
-      <cylinder_inertia m="5" r="0.1" h="0.05"/>
-      <inertia
-        ixx="1.0" ixy="0.0" ixz="0.0"
-        iyy="1.0" iyz="0.0"
-        izz="1.0"/>
-    </inertial>
-  </link>
-  <joint type="continuous" name="left_wheel_hinge">
-    <origin xyz="0.1 0.15 0" rpy="0 0 0"/>
-    <child link="left_wheel"/>
-    <parent link="chassis"/>
-    <axis xyz="0 1 0" rpy="0 0 0"/>
-    <limit effort="100" velocity="100"/>
-    <joint_properties damping="0.0" friction="0.0"/>
-  </joint>
-  <joint type="continuous" name="right_wheel_hinge">
-    <origin xyz="0.1 -0.15 0" rpy="0 0 0"/>
-    <child link="right_wheel"/>
-    <parent link="chassis"/>
-    <axis xyz="0 1 0" rpy="0 0 0"/>
-    <limit effort="100" velocity="100"/>
-    <joint_properties damping="0.0" friction="0.0"/>
-  </joint>
+    <xacro:include filename="$(find mybot_description)/urdf/mybot.gazebo" />
+    <link name="chassis">
+      <inertial>
+        <mass value="2.0"/>
+        <origin rpy="0 0 0" xyz="0 0 0"/>
+        <inertia ixx="0.08025" ixy="0" ixz="0"
+                 iyy="0.08025" iyz="0"
+                 izz="0.1445"
+        />
+      </inertial>
+      <collision>
+        <origin rpy="1.57079632679 0.0 1.57079632679" xyz="0.0 0.0 0.086"/>
+        <geometry>
+          <mesh filename="file://$(find mybot_description)/meshes/*.dae file" scale="0.002 0.002 0.002"/>
+        </geometry>
+      </collision>
+      <visual>
+        <origin rpy="1.57079632679 0.0 1.57079632679" xyz="0.0 0.0 0.086"/>
+        <geometry>
+          <mesh filename="file://$(find mybot_description)/meshes/*.dae file" scale="0.002 0.002 0.002"/>
+        </geometry>
+      </visual>
+    </link>
+    <link name="left_wheel">
+      <inertial>
+        <mass value="0.3"/>
+        <origin rpy="0 0 0" xyz="0 0 0"/>
+        <inertia ixx="0.000129167" ixy="0" ixz="0"
+                 iyy="0.000129167" iyz="0"
+                 izz="0.0000225"
+        />
+      </inertial>
+      <collision>
+        <origin rpy="0 0 0" xyz="0 0 0"/>
+        <geometry>
+          <mesh filename="file://$(find mybot_description)/meshes/*.dae file" scale="0.002 0.002 0.002"/>
+        </geometry>
+      </collision>
+      <visual>
+        <origin rpy="0 0 0" xyz="0 0 0"/>
+          <geometry>
+            <mesh filename="file://$(find mybot_description)/meshes/*.dae file" scale="0.002 0.002 0.002"/>
+          </geometry>
+      </visual>
+    </link>
+    <joint name='left_wheel_hinge' type='revolute'>
+      <origin rpy="0.0 0.0 1.57079632679" xyz="0.06 0.1025 0.06"/>
+      <child  link="left_wheel"/>
+      <parent link="chassis"/>
+      <axis rpy="0 0 0" xyz="1 0 0"/>
+      <limit lower="-1e+16" upper="1e+16" effort="100" velocity="100"/>
+    </joint>
+    <link name="right_wheel">
+      <inertial>
+        <mass value="0.3"/>
+        <origin rpy="0 0 0" xyz="0 0 0"/>
+        <inertia ixx="0.000129167" ixy="0" ixz="0"
+                 iyy="0.000129167" iyz="0"
+                 izz="0.0000225"
+        />
+      </inertial>
+      <collision>
+        <origin rpy="0 0 0" xyz="0 0 0"/>
+        <geometry>
+          <mesh filename="file://$(find mybot_description)/meshes/*.dae file" scale="0.002 0.002 0.002"/>
+        </geometry>
+      </collision>
+      <visual>
+        <origin rpy="0 0 0" xyz="0 0 0"/>
+        <geometry>
+          <mesh filename="file://$(find mybot_description)/meshes/*.dae file" scale="0.002 0.002 0.002"/>
+        </geometry>
+      </visual>
+    </link>
+    <joint name='right_wheel_hinge' type='revolute'>
+      <origin rpy="0.0 0.0 1.57079632679 " xyz="0.06 -0.119 0.06"/>
+      <child  link="right_wheel"/>
+      <parent link="chassis"/>
+      <axis rpy="0 0 0" xyz="1 0 0"/>
+      <limit lower="-1e+16" upper="1e+16" effort="100" velocity="100"/>
+    </joint>
 </robot>
